Commit message: updated hippo and thruster parameters

File: models/hippo3/urdf/hippo3_params.xacro (robot description, xacro)
@@ -1,9 +1,9 @@
 <?xml version="1.0"?>
 <robot xmlns:xacro="http://www.ros.org/wiki/xacro">
-    <xacro:property name="base_mass" value="2.31" />
-    <xacro:property name="ixx" value="0.0024" />
-    <xacro:property name="iyy" value="0.010717" />
-    <xacro:property name="izz" value="0.010717" />
-    <xacro:property name="thruster_r" value="0.097" />
+    <xacro:property name="base_mass" value="2.655" />
+    <xacro:property name="ixx" value="0.007" />
+    <xacro:property name="iyy" value="0.028" />
+    <xacro:property name="izz" value="0.028" />
+    <xacro:property name="thruster_r" value="0.06" />
     <xacro:property name="added_mass_linear" value="1.11 2.8 2.8" />
     <xacro:property name="added_mass_angular" value="0.00451 0.0163 0.0163"/>

File: models/thruster/urdf/thruster_params.xacro (robot description, xacro)
@@ -5,12 +5,12 @@
     <xacro:property name="thruster_iyy" value="1e-6" />
     <xacro:property name="thruster_izz" value="1e-6" />
-    <xacro:property name="thrust_quadratic_coeff" value="3.313e-3" />
-    <xacro:property name="thrust_linear_coeff" value="0.1086" />
-    <xacro:property name="thrust_constant_coeff" value="-0.8576" />
+    <xacro:property name="thrust_quadratic_coeff" value="0.00283" />
+    <xacro:property name="thrust_linear_coeff" value="0.0911" />
+    <xacro:property name="thrust_constant_coeff" value="-0.005" />
     <!-- Throttle = f(revs/s) -->
     <xacro:property name="velocity_quadratic_coeff" value="1.2679e-4"/>
     <xacro:property name="velocity_linear_coeff" value="1.1105e-2"/>
     <xacro:property name="velocity_constant_coeff" value="0.0"/>
-    <xacro:property name="torque_constant" value="1e-2" />
+    <xacro:property name="torque_constant" value="0.0092" />
     <xacro:property name="rpm_scaler" value="1" />
     <xacro:property name="max_rpm" value="3000" />
