Commit message: updated time constant for thruster dynamics from experiemntal data

File: models/thruster/urdf/thruster_params.xacro (robot description, xacro)
@@ -15,6 +15,6 @@
     <xacro:property name="rpm_scaler" value="1" />
     <xacro:property name="max_rpm" value="3000" />
-    <xacro:property name="timeconstant_up" value="0.00" />
-    <xacro:property name="timeconstant_down" value="0.00" />
+    <xacro:property name="timeconstant_up" value="0.4" />
+    <xacro:property name="timeconstant_down" value="0.4" />
     <xacro:property name="propeller_mesh" value="$(find hippo_sim)/models/thruster/meshes/propeller.dae" />
 </robot>

Commit message: updated thruster time constant after experimental transient analysis

File: models/thruster/urdf/thruster_params.xacro (robot description, xacro)
@@ -15,6 +15,6 @@
     <xacro:property name="rpm_scaler" value="1" />
     <xacro:property name="max_rpm" value="3000" />
-    <xacro:property name="timeconstant_up" value="0.4" />
-    <xacro:property name="timeconstant_down" value="0.4" />
+    <xacro:property name="timeconstant_up" value="0.2" />
+    <xacro:property name="timeconstant_down" value="0.2" />
     <xacro:property name="propeller_mesh" value="$(find hippo_sim)/models/thruster/meshes/propeller.dae" />
 </robot>
